Commit message: Son 19/10/2023

File: urdf/mvibot3.urdf (robot description, URDF)
Before this commit: robot mvibot, 8 links, 7 joints
Links:
- link $(arg mvibot_seri)/base_link: geometry visual mesh filename=file:///home/hitech/catkin_ws/src/mvibot_v4/urdf/dir3.stl scale=0.001 0.001 0.001; visual mesh filename=file:///home/hitech/catkin_ws/src/mvibot_v4/urdf/mvibot5.stl scale=0.001 0.001 0.001

File: urdf/mvibot_web.urdf (robot description, URDF)
Before this commit: robot mvibot, 1 links, 0 joints
Links:
- link $(arg mvibot_seri)/base_footprint: geometry visual mesh filename=dir3.stl scale=0.001 0.001 0.001; visual mesh filename=mvibot5.stl scale=0.001 0.001 0.001
